File: Hardware/PCB/GPS/GPS.kicad_pcb (KiCad board)
At the start: 2 copper layers, 25.2 x 30.5 mm, 12 parts, among them J1 Conn_01x06_Socket, U1 SAM-M10Q-00B, U2 AMS1117-3.3, U3 IST8310

Commit message: Gps update
Parts:
- removed C3: 4.7uF, Capacitor_SMD:C_0603_1608Metric
- removed C5, C6: 0.1uF, Capacitor_SMD:C_0603_1608Metric
- removed U3: IST8310, Package_LGA:LGA-16_3x3mm_P0.5mm
- added C7: 10uf, Capacitor_SMD:C_0603_1608Metric, F.Cu at (113.9, 81.5)
- added C8: 1 uf, Capacitor_SMD:C_0603_1608Metric, F.Cu at (112.7, 76.7)
- added U4: MMC5983MA, Compass:MMC5983MA_MEM, F.Cu at (110.0, 80.3)
- moved C2 2.40 mm to (114.7, 79.2), turned to -90 degrees
- moved R1 2.03 mm to (108.9, 76.7), turned to -90 degrees
Connections:
- net /3v3 renamed 3v3
- net /gnd renamed gnd
Routing:
- net 3v3: track 105.9 -> 100.8 mm, vias 5 -> 2
- net Net-(U4-CAP): track 0.00 -> 2.20 mm
- net /gps_c1: track 1.96 -> 0.00 mm
- net /comp_sda: track 50.2 -> 48.8 mm
- net /comp_scl: track 49.5 -> 49.0 mm
