File: Hardware/PCB/GPS/Old/GPS.kicad_sch (KiCad schematic)
At the start: 11 parts, among them J1 Conn_01x06_Socket, U1 SAM-M10Q-00B, U2 AMS1117-3.3, U4 MMC5983MA

Commit message: Gps update
Parts:
- removed C7: 10uf, Capacitor_SMD:C_0603_1608Metric, symbol Device:C
- removed C8: 1 uf, Capacitor_SMD:C_0603_1608Metric, symbol Device:C
- removed U4: MMC5983MA, Compass:MMC5983MA_MEM, symbol MMC5983MA:MMC5983MA
- added C3: 4.7uF, Capacitor_SMD:C_0603_1608Metric, symbol Device:C
- added C5, C6: 0.1uF, Capacitor_SMD:C_0603_1608Metric, symbol Device:C
- added U3: IST8310, Package_LGA:LGA-16_3x3mm_P0.5mm, symbol Sensor_Magnetic:IST8310
Connections:
- net 3v3: now also C5.2, C6.2, U3.13 (DVDD), U3.2 (AVDD)
- net comp_scl: now also U3.1 (SCL)
- net comp_sda: now also U3.16 (SDA)
- net gnd: now also C3.2, C5.1, C6.1, U3.11 (VSS), U3.5 (CAD0), U3.6 (CAD1), U3.9 (VSS)
- new net gps_c1: C3.1, U3.10 (C1)
- no-connect marks 9 -> 10
