File: archive/Payload_PCB.kicad_pcb (KiCad board)
At the start: 2 copper layers, 40 x 22.5 mm, 16 parts, among them J1 PI IN, J2 USB_C_Receptacle_USB2.0_16P, J3 payload out, J4 nfc, Q1 AO3400A, U1 ESP32-S3-MINI-1U, U2 AP63203WU

Commit message: Payload update
Parts:
- L1: footprint Inductor_SMD:L_1008_2520Metric -> Inductor_SMD:L_0603_1608Metric
- moved L1 0.63 mm to (153.2, 109.0)
- moved C3 0.43 mm to (153.2, 106.6)
Routing:
- net /+3v3: track 21.1 -> 20.4 mm
Changed lines of the file:
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@@
 			(drillshape 0)
 			(scaleselection 1)
-			(outputdirectory "Production_v2/")
+			(outputdirectory "")
 		)
 	)
@@
 		(property ki_fp_filters "R_*")
 		(sheetname "/")
-		(sheetfile "Payload_PCB.kicad_sch")
+		(sheetfile "AHHHHHH.kicad_sch")
 		(units
 			(unit
@@
 	(footprint "Capacitor_SMD:C_0603_1608Metric"
 		(layer "F.Cu")
-		(at 153.16 106.17 180)
+		(at 153.225 106.6 180)
 		(descr "Capacitor SMD 0603 (1608 Metric), square (rectangular) end terminal, IPC-7351 nominal, (Body size source: IPC-SM-782 page 76, https://www.pcb-3d.com/wordpress/wp-content/uploads/ipc-sm-782a_amendment_1_and_2.pdf)")
 		(tags "capacitor")
@@
 		(property ki_fp_filters "C_*")
 		(sheetname "/")
-		(sheetfile "Payload_PCB.kicad_sch")
+		(sheetfile "AHHHHHH.kicad_sch")
 		(units
 			(unit
@@
 		(property ki_fp_filters "C_*")
 		(sheetname "/")
-		(sheetfile "Payload_PCB.kicad_sch")
+		(sheetfile "AHHHHHH.kicad_sch")
 		(units
 			(unit
@@
 		(property ki_fp_filters "Connector*:*_1x??_*")
 		(sheetname "/")
-		(sheetfile "Payload_PCB.kicad_sch")
+		(sheetfile "AHHHHHH.kicad_sch")
 		(units
 			(unit
@@
 		(property ki_fp_filters "TSOT?23*")
 		(sheetname "/")
-		(sheetfile "Payload_PCB.kicad_sch")
+		(sheetfile "AHHHHHH.kicad_sch")
 		(units
 			(unit
@@
 		(property ki_fp_filters "R_*")
 		(sheetname "/")
-		(sheetfile "Payload_PCB.kicad_sch")
+		(sheetfile "AHHHHHH.kicad_sch")
 		(units
 			(unit
@@
 		(property ki_fp_filters "Connector*:*_1x??_*")
 		(sheetname "/")
-		(sheetfile "Payload_PCB.kicad_sch")
+		(sheetfile "AHHHHHH.kicad_sch")
 		(units
 			(unit
@@
 		(property ki_fp_filters "D*SMA*")
 		(sheetname "/")
-		(sheetfile "Payload_PCB.kicad_sch")
+		(sheetfile "AHHHHHH.kicad_sch")
 		(units
 			(unit
@@
 		(property ki_fp_filters "Connector*:*_1x??_*")
 		(sheetname "/")
-		(sheetfile "Payload_PCB.kicad_sch")
+		(sheetfile "AHHHHHH.kicad_sch")
 		(units
 			(unit
@@
 		(property ki_fp_filters "C_*")
 		(sheetname "/")
-		(sheetfile "Payload_PCB.kicad_sch")
+		(sheetfile "AHHHHHH.kicad_sch")
 		(units
 			(unit
@@
 		(property ki_fp_filters "R_*")
 		(sheetname "/")
-		(sheetfile "Payload_PCB.kicad_sch")
+		(sheetfile "AHHHHHH.kicad_sch")
 		(units
 			(unit
@@
 		)
 	)
-	(footprint "Inductor_SMD:L_1008_2520Metric"
+	(footprint "Inductor_SMD:L_0603_1608Metric"
 		(layer "F.Cu")
-		(at 153.11 108.38)
-		(descr "Inductor SMD 1008 (2520 Metric), square (rectangular) end terminal, IPC-7351 nominal, (Body size source: https://ecsxtal.com/store/pdf/ECS-MPI2520-SMD-POWER-INDUCTOR.pdf)")
+		(at 153.2125 109)
+		(descr "Inductor SMD 0603 (1608 Metric), square (rectangular) end terminal, IPC-7351 nominal, (Body size source: http://www.tortai-tech.com/upload/download/2011102023233369053.pdf)")
 		(tags "inductor")
 		(property "Reference" "L1"
-			(at 0 -2.05 0)
+			(at 0 -1.43 0)
 			(layer "F.SilkS")
+			(hide yes)
 			(effects
 				(font
@@
 		)
 		(property "Value" "2.2 uH"
-			(at 0 2.05 0)
+			(at 0 1.43 0)
 			(layer "F.Fab")
+			(hide yes)
 			(effects
 				(font
@@
 		(property ki_fp_filters "Choke_* *Coil* Inductor_* L_*")
 		(sheetname "/")
-		(sheetfile "Payload_PCB.kicad_sch")
+		(sheetfile "AHHHHHH.kicad_sch")
 		(units
 			(unit
@@
 		(duplicate_pad_numbers_are_jumpers no)
 		(fp_line
-			(start -0.261252 -1.11)
-			(end 0.261252 -1.11)
+			(start -0.162779 -0.51)
+			(end 0.162779 -0.51)
 			(stroke
 				(width 0.12)
@@
 		)
 		(fp_line
-			(start -0.261252 1.11)
-			(end 0.261252 1.11)
+			(start -0.162779 0.51)
+			(end 0.162779 0.51)
 			(stroke
 				(width 0.12)
@@
 		)
 		(fp_rect
-			(start -1.95 -1.35)
-			(end 1.95 1.35)
+			(start -1.48 -0.73)
+			(end 1.48 0.73)
 			(stroke
 				(width 0.05)
@@
 		)
 		(fp_rect
-			(start -1.25 -1)
-			(end 1.25 1)
+			(start -0.8 -0.4)
+			(end 0.8 0.4)
 			(stroke
 				(width 0.1)
@@
 			(effects
 				(font
-					(size 0.62 0.62)
-					(thickness 0.09)
+					(size 0.4 0.4)
+					(thickness 0.06)
 				)
 			)
 		)
 		(pad "1" smd roundrect
-			(at -1.075 0)
-			(size 1.25 2.2)
+			(at -0.7875 0)
+			(size 0.875 0.95)
 			(layers "F.Cu" "F.Mask" "F.Paste")
-			(roundrect_rratio 0.2)
+			(roundrect_rratio 0.25)
 			(net "/sw")
 			(pinfunction "1_1")
@@
 		)
 		(pad "2" smd roundrect
-			(at 1.075 0)
-			(size 1.25 2.2)
+			(at 0.7875 0)
+			(size 0.875 0.95)
 			(layers "F.Cu" "F.Mask" "F.Paste")
-			(roundrect_rratio 0.2)
+			(roundrect_rratio 0.25)
 			(net "/+3v3")
 			(pinfunction "2_2")
@@
 		)
 		(embedded_fonts no)
-		(model "${KICAD10_3DMODEL_DIR}/Inductor_SMD.3dshapes/L_1008_2520Metric.step"
+		(model "${KICAD10_3DMODEL_DIR}/Inductor_SMD.3dshapes/L_0603_1608Metric.step"
 			(offset
 				(xyz 0 0 0)
@@
 		(property ki_fp_filters "ESP32?S*MINI?1U")
 		(sheetname "/")
-		(sheetfile "Payload_PCB.kicad_sch")
+		(sheetfile "AHHHHHH.kicad_sch")
 		(units
 			(unit
@@
 		(property ki_fp_filters "SOT?23*")
 		(sheetname "/")
-		(sheetfile "Payload_PCB.kicad_sch")
+		(sheetfile "AHHHHHH.kicad_sch")
 		(units
 			(unit
@@
 		(property ki_fp_filters "USB*C*Receptacle*")
 		(sheetname "/")
-		(sheetfile "Payload_PCB.kicad_sch")
+		(sheetfile "AHHHHHH.kicad_sch")
 		(units
 			(unit
@@
 			(at 0 -1.448 0)
 			(layer "F.SilkS")
-			(hide yes)
 			(effects
 				(font
@@
 		(property ki_fp_filters "Pin* Test*")
 		(sheetname "/")
-		(sheetfile "Payload_PCB.kicad_sch")
+		(sheetfile "AHHHHHH.kicad_sch")
 		(units
 			(unit
@@
 	)
 	(segment
-		(start 153.935 106.17)
-		(end 153.935 106.075)
-		(width 0.5)
-		(layer "F.Cu")
-		(net "/+3v3")
-	)
-	(segment
-		(start 151.525 116.025)
-		(end 151.6 116.1)
-		(width 0.5)
-		(layer "F.Cu")
-		(net "/+3v3")
-	)
-	(segment
-		(start 153.935 106.075)
-		(end 155.39 104.62)
+		(start 154 109)
+		(end 154 106.6)
 		(width 0.5)
 		(layer "F.Cu")
@@
 	)
 	(segment
-		(start 155.35 106.4)
-		(end 155.12 106.17)
+		(start 154 106.6)
+		(end 155.55 105.05)
 		(width 0.5)
 		(layer "F.Cu")
@@
 	)
 	(segment
-		(start 151.525 114.8)
-		(end 151.525 116.025)
+		(start 155.35 109)
+		(end 155.35 107.45)
 		(width 0.5)
 		(layer "F.Cu")
@@
 	)
 	(segment
-		(start 155.35 109)
-		(end 155.35 106.4)
+		(start 151.525 116.025)
+		(end 151.6 116.1)
 		(width 0.5)
 		(layer "F.Cu")
@@
 	)
 	(segment
-		(start 154.185 108.38)
-		(end 154.185 106.42)
+		(start 154.5 106.6)
+		(end 155.35 107.45)
 		(width 0.5)
 		(layer "F.Cu")
@@
 	)
 	(segment
-		(start 155.12 106.17)
-		(end 153.935 106.17)
+		(start 151.525 114.8)
+		(end 151.525 116.025)
 		(width 0.5)
 		(layer "F.Cu")
@@
 	)
 	(segment
-		(start 154.185 106.42)
-		(end 153.935 106.17)
+		(start 154 106.6)
+		(end 154.5 106.6)
 		(width 0.5)
 		(layer "F.Cu")
@@
 	)
 	(segment
-		(start 151.37 106.17)
-		(end 151.17 106.37)
-		(width 0.25)
-		(layer "F.Cu")
-		(net "/gnd")
-	)
-	(segment
 		(start 171.25 117.65)
 		(end 171.25 119.15)
@@
 	)
 	(segment
+		(start 152.45 106.6)
+		(end 151.5 106.6)
+		(width 0.2)
+		(layer "F.Cu")
+		(net "/gnd")
+	)
+	(segment
 		(start 168.75 99.95)
 		(end 169.05 100.25)
@@
 	)
 	(segment
-		(start 152.385 106.17)
-		(end 151.37 106.17)
-		(width 0.25)
-		(layer "F.Cu")
-		(net "/gnd")
-	)
-	(segment
 		(start 162.6 110.65)
 		(end 165.9 110.65)
@@
 	)
 	(segment
+		(start 151.5 106.6)
+		(end 151.1 107)
+		(width 0.2)
+		(layer "F.Cu")
+		(net "/gnd")
+	)
+	(segment
 		(start 171.25 119.15)
 		(end 171.3 119.2)
@@
 	)
 	(via
-		(at 151.17 106.37)
-		(size 0.6)
-		(drill 0.3)
-		(layers "F.Cu" "B.Cu")
-		(net "/gnd")
-	)
-	(via
 		(at 162.6 107.6)
 		(size 0.6)
@@
 	)
 	(via
+		(at 151.1 107)
+		(size 0.6)
+		(drill 0.3)
+		(layers "F.Cu" "B.Cu")
+		(net "/gnd")
+	)
+	(via
 		(at 171.3 119.2)
 		(size 0.6)
@@
 		(polygon
 			(pts
-				(xy 155.686273 105.36442) (xy 155.65 115.35) (xy 154.65 116.45) (xy 151.25 116.45) (xy 151.2 115.8)
-				(xy 154.2 115.75) (xy 154.95 114.9) (xy 154.915386 109.880934) (xy 153.559194 109.899138) (xy 153.394936 105.448995)
+				(xy 155.7 107.2) (xy 155.65 115.35) (xy 154.65 116.45) (xy 151.25 116.45) (xy 151.2 115.8) (xy 154.2 115.75)
+				(xy 154.95 114.9) (xy 154.9 107.65) (xy 154.65 107.45) (xy 154.65 106.15)
 			)
 		)
