File: Hardware/PCB/Flight_Controller/HermesFC.kicad_sch (KiCad schematic)
At the start: 0 parts

Commit message: FC update
Other:
- company: (none) -> Aadil Naji
- title: (none) -> Hermes Flight Controller
Changed lines of the file:
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@@
 	(paper "A4")
 	(title_block
-		(date "23/4/2026")
+		(title "Hermes Flight Controller")
+		(date "2025-03-12")
 		(rev "v1.0")
+		(company "Aadil Naji")
+		(comment 1 "HERMESFLIGHT CONTROLLER V1.0")
 	)
 	(sheet
@@
 		)
 		(instances
-			(project "Streetsafe"
+			(project "HermesFC"
 				(path "/7c1ac307-4d35-4291-88c2-548b52d0f9f3"
 					(page "2")
@@
 		)
 		(instances
-			(project "Streetsafe"
+			(project "HermesFC"
 				(path "/7c1ac307-4d35-4291-88c2-548b52d0f9f3"
 					(page "3")
